File: Keres.kicad_sch (KiCad schematic)
At the start: 7 parts, among them J1 XT90M, J2 DSUB44S_HD, J4 2.54mm Pin Header

Commit message: Update BOM, Gerber Outputs, Fiducials
Parts:
- added FID1, FID2, FID3, FID4, FID5, FID6: Fiducial, Fiducial:Fiducial_0.75mm_Mask1.5mm, symbol Mechanical:Fiducial
- J1: MPN (none) -> XT90PW; Manufacturer (none) -> ELFCULB; now not fitted
- J2: MPN (none) -> 10090926-P444XLF; Manufacturer (none) -> Amphenol ICC (FCI)
- J4: MPN (none) -> 0022285034; Manufacturer (none) -> Molex
