File: Microcontroller.kicad_sch (KiCad schematic)
At the start: 42 parts, among them J3 U_FL-R-SMT-1_10_, U5 BMP280, U6 MAX-M10S, U7 Teensy 4.0, U8 MPU-6050

Commit message: Update PCBA Layout
Redo full PCBA layout
Connections:
- net ESC1_EN: now also U7.15 (13); no longer U7.2 (0)
- net ESC2_EN: now also U7.2 (0); no longer U7.13 (11)
- net ESC3_EN: now also U7.13 (11); no longer U7.14 (12)
- net ESC4_EN: now also U7.14 (12); no longer U7.15 (13)
Changed lines of the file:
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@@
-		)
-	)
-	(label "ESC3_EN"
-		(at 100.33 140.97 0)
-		(effects
-			(font
-				(size 1.27 1.27)
-			)
-			(justify left bottom)
-		)
-	)
-	(label "ESC4_EN"
-		(at 184.15 144.78 180)
-		(effects
-			(font
-				(size 1.27 1.27)
-			)
-			(justify right bottom)
 		)
 	)
@@
 		)
 	)
-	(label "ESC2_EN"
-		(at 100.33 138.43 0)
-		(effects
-			(font
-				(size 1.27 1.27)
-			)
-			(justify left bottom)
-		)
-	)
 	(label "SCL_1"
 		(at 187.96 125.73 180)
@@
 		)
 	)
+	(label "ESC2_EN"
+		(at 100.33 105.41 0)
+		(effects
+			(font
+				(size 1.27 1.27)
+			)
+			(justify left bottom)
+		)
+	)
+	(label "ESC4_EN"
+		(at 100.33 140.97 0)
+		(effects
+			(font
+				(size 1.27 1.27)
+			)
+			(justify left bottom)
+		)
+	)
 	(label "PWM_ESC3"
 		(at 100.33 113.03 0)
@@
 		)
 	)
-	(label "ESC1_EN"
-		(at 100.33 105.41 0)
-		(effects
-			(font
-				(size 1.27 1.27)
-			)
-			(justify left bottom)
-		)
-	)
 	(label "PWM_SRVO3"
 		(at 232.41 116.84 0)
@@
 		)
 	)
+	(label "ESC3_EN"
+		(at 100.33 138.43 0)
+		(effects
+			(font
+				(size 1.27 1.27)
+			)
+			(justify left bottom)
+		)
+	)
 	(label "ESC2_EN"
 		(at 232.41 82.55 0)
@@
 		)
 	)
+	(label "ESC1_EN"
+		(at 184.15 144.78 180)
+		(effects
+			(font
+				(size 1.27 1.27)
+			)
+			(justify right bottom)
+		)
+	)

Commit message: Update BOM, Gerber Outputs, Fiducials
Parts:
- C16, C17, C18, C19, C21, C22, C23: MPN (none) -> C0603C104K5RACAUTO; Manufacturer (none) -> Kemet
- C20: MPN (none) -> C0603C103K5RACAUTO; Manufacturer (none) -> Kemet
- C24: MPN (none) -> C0603C222K5RACAUTO; Manufacturer (none) -> Kemet
- D9: MPN (none) -> LTST-C190KSKT; Manufacturer (none) -> Lite-On Inc.
- J3: MPN (none) -> U.FL-R-SMT-1(10); Manufacturer (none) -> Hirose Electric Co Ltd
- L3: MPN (none) -> LQG18HN27NJ00; Manufacturer (none) -> Murata Electronics
- R12, R31, R34, R35, R37, R38, R74, R75, R76, R77: MPN (none) -> CRCW06030000Z0EA; Manufacturer (none) -> Vishay Dale
- R20: MPN (none) -> CRCW060310R0FKEA; Manufacturer (none) -> Vishay Dale
- R21, R23, R25, R29, R30, R32, R33: MPN (none) -> CRCW060310K0FKEA; Manufacturer (none) -> Vishay Dale
- U6: MPN (none) -> MAX-M10S; Manufacturer (none) -> u-blox
- U7: MPN (none) -> 4.0 Microcontroller; Manufacturer (none) -> Teensy; now not fitted
- U8: MPN (none) -> MPU-6050; Manufacturer (none) -> TDK InvenSense
