File: Power.kicad_sch (KiCad schematic)
At the start: 61 parts, among them Q1 SiS443DN, Q2 SQJQ116EL, Q3 SQJQ116EL, Q4 SQJQ116EL, Q5 SQJQ116EL, U1 TLV76133DCY, U2 LM22678TJ-5, U3 LM22678TJ-5, U4 LM22678TJ-5

Commit message: Update BOM, Gerber Outputs, Fiducials
Parts:
- C1, C2: MPN (none) -> T491X226K050ATAUTO; Manufacturer (none) -> Kemet
- C10, C15, C38, C4, C5, C6: MPN (none) -> 0603X7R105KT1AT; Manufacturer (none) -> KYOCERA AVX; now left out of the parts list
- C11, C3, C34: MPN (none) -> C0603C103K5RACAUTO; Manufacturer (none) -> Kemet
- C12, C13, C35, C36, C7, C8: MPN (none) -> TAJC476K016RNJ; Manufacturer (none) -> KYOCERA AVX; now left out of the parts list
- C14, C37, C9: MPN (none) -> 0603DD106MAT2A; Manufacturer (none) -> KYOCERA AVX
- D1: MPN (none) -> BZV55B16; Manufacturer (none) -> Taiwan Semiconductor Corporation
- D11, D4, D5, D6: MPN (none) -> LTST-C190KGKT; Manufacturer (none) -> Lite-On Inc.
- D2, D3: MPN (none) -> SMAJ40A; Manufacturer (none) -> Littelfuse Inc.
- L1, L2, L4: MPN (none) -> XAL1010-682MED; Manufacturer (none) -> Coilcraft
- Q1: MPN (none) -> SIS443DN-T1-GE3; Manufacturer (none) -> Vishay Siliconix
- Q2, Q3, Q4, Q5: MPN (none) -> SQJQ116EL-T1_GE3; Manufacturer (none) -> Vishay Semiconductors
- R1, R10, R6, R8: MPN (none) -> CSS4J-4026R-L300F; Manufacturer (none) -> Bourns Inc.
- R11, R3, R4: MPN (none) -> CRCW060312K7FKEA; Manufacturer (none) -> Vishay Dale
- R13, R67, R68: MPN (none) -> ERJ-U120R00U; Manufacturer (none) -> Panasonic Industry
- R16, R17, R18, R19: MPN (none) -> CRCW06031K00FKEA; Manufacturer (none) -> Vishay Dale
- R2: MPN (none) -> CRCW060310K0FKEA; Manufacturer (none) -> Vishay Dale
- R5, R9: MPN (none) -> CRCW080510K0FKEA; Manufacturer (none) -> Vishay Dale
- R7: MPN (none) -> BVT-I-R005-1.0; Manufacturer (none) -> Isabellenhuette USA
- U1: MPN (none) -> TLV76133DCYR; Manufacturer (none) -> Texas Instruments
- U2, U3, U4: MPN (none) -> LM22678TJ-5.0/NOPB; Manufacturer (none) -> Texas Instruments
